File: pcbs/matrix-right/matrix-right.kicad_sch (KiCad schematic)
At the start: 51 parts, among them J4 Conn_01x11, SW1 SW_Push, SW10 SW_Push, SW11 SW_Push, SW12 SW_Push, SW13 SW_Push, SW14 SW_Push, SW15 SW_Push, SW16 SW_Push, SW17 SW_Push, SW18 SW_Push, SW19 SW_Push, SW2 SW_Push, SW20 SW_Push, SW21 SW_Push, SW22 SW_Push, SW23 SW_Push, SW24 SW_Push, SW25 SW_Push, SW3 SW_Push, SW4 SW_Push, SW5 SW_Push, SW6 SW_Push, SW7 SW_Push, SW8 SW_Push, SW9 SW_Push

Commit message: Assign the matrix J1 pins per side to match the routing
Order the J1 pins so each net leaves toward its destination (columns
C0-C3 on one side, C5-C6 on the other, rows above and below), mirrored
between the halves:
  left  (pin 11..1): C3 C2 C1 C0 R3 R2 R1 R0 C4 C6 C5
  right (pin 11..1): C5 C6 R3 R2 R1 R0 C4 C0 C1 C2 C3
The controller board and cable are unchanged; with matrix pin k on
controller pin 12 - k, the XIAO pins become
  left:  C0-C6 = D3 D4 D5 D6 D9 D7 D8, R0-R3 = D10 D0 D1 D2
  right: C0-C6 = D10 D9 D8 D7 D0 D6 D5, R0-R3 = D1 D2 D3 D4
Split the root project's shared matrix sheet into left and right copies.

Co-Authored-By: Claude Opus 5.5 <noreply@anthropic.com>
Connections:
- net C0: now also J4.4 (Pin_4); no longer J4.5 (Pin_5)
- net C1: now also J4.3 (Pin_3); no longer J4.6 (Pin_6)
- net C2: now also J4.2 (Pin_2); no longer J4.7 (Pin_7)
- net C3: now also J4.1 (Pin_1); no longer J4.8 (Pin_8)
- net C4: now also J4.5 (Pin_5); no longer J4.9 (Pin_9)
- net C5: now also J4.11 (Pin_11); no longer J4.10 (Pin_10)
- net C6: now also J4.10 (Pin_10); no longer J4.11 (Pin_11)
- net R0: now also J4.6 (Pin_6); no longer J4.1 (Pin_1)
- net R1: now also J4.7 (Pin_7); no longer J4.2 (Pin_2)
- net R2: now also J4.8 (Pin_8); no longer J4.3 (Pin_3)
- net R3: now also J4.9 (Pin_9); no longer J4.4 (Pin_4)
Changed lines of the file:
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@@
 		)
 	)
-	(label "C0"
+	(label "C4"
 		(at 229.87 43.18 0)
 		(effects
@@
 		)
 	)
-	(label "R1"
+	(label "C2"
 		(at 229.87 35.56 0)
 		(effects
@@
 		)
 	)
-	(label "C2"
+	(label "R1"
 		(at 229.87 48.26 0)
 		(effects
@@
 		)
 	)
-	(label "C4"
+	(label "R3"
 		(at 229.87 53.34 0)
 		(effects
@@
 		)
 	)
-	(label "R3"
+	(label "C0"
 		(at 229.87 40.64 0)
 		(effects
@@
 		)
 	)
-	(label "C6"
+	(label "C5"
 		(at 229.87 58.42 0)
 		(effects
@@
 		)
 	)
-	(label "C3"
+	(label "R2"
 		(at 229.87 50.8 0)
 		(effects
@@
 		)
 	)
-	(label "R0"
+	(label "C3"
 		(at 229.87 33.02 0)
 		(effects
@@
 		)
 	)
-	(label "R2"
+	(label "C1"
 		(at 229.87 38.1 0)
 		(effects
@@
 		)
 	)
-	(label "C1"
+	(label "R0"
 		(at 229.87 45.72 0)
 		(effects
@@
 		)
 	)
-	(label "C5"
+	(label "C6"
 		(at 229.87 55.88 0)
 		(effects

Commit message: Add LCSC part numbers to the matrix boards
Run add_lcsc_fields.py on the matrix schematics (and the root copies)
and update both boards from the schematic, so the footprints carry the
LCSC field too. Nothing else changes on the boards.

Co-Authored-By: Claude Opus 5.5 <noreply@anthropic.com>
Parts:
- D1, D10, D11, D12, D13, D14, D15, D16, D17, D18, D19, D2, D20, D21, D22, D23, D24, D25, D3, D4, D5, D6, D7, D8, D9: LCSC (none) -> C81598
- J4: LCSC (none) -> C515956
- SW1, SW10, SW11, SW12, SW13, SW14, SW15, SW16, SW17, SW18, SW19, SW2, SW20, SW21, SW22, SW23, SW24, SW25, SW3, SW4, SW5, SW6, SW7, SW8, SW9: LCSC (none) -> C41430893
